Commit message: Day 2 complete - warehouse with aisles, lidar URDF, A* integration tested

File: description/robot.urdf.xacro (robot description, xacro)
@@ -1,4 +1,5 @@
 <?xml version="1.0"?>
 <robot xmlns:xacro="http://www.ros.org/wiki/xacro" name="warehouse_robot">
+  <!-- Properties -->
   <xacro:property name="body_length"  value="0.6"/>
   <xacro:property name="body_width"   value="0.4"/>
@@ -8,4 +9,5 @@
   <xacro:property name="wheel_x"      value="0.15"/>
   <xacro:property name="wheel_y"      value="0.225"/>
+  <!-- Materials -->
   <material name="grey">
     <color rgba="0.5 0.5 0.5 1"/>
@@ -20,34 +22,37 @@
     <color rgba="0.1 0.1 0.1 1"/>
   </material>
-    <link name="base_link"/>
-    <joint name="chassis_joint" type="fixed">
-      <parent link="base_link"/>
-      <child link="chassis"/>
-      <origin xyz="0 0 0.2"/>
-    </joint>
-    <link name="chassis">
-      <visual>
-        <origin xyz="0 0 0"/>
-        <geometry>
-          <box size="${body_length} ${body_width} ${body_height}"/>
-        </geometry>
-        <material name="grey"/>
-      </visual>
-      <collision>
-        <origin xyz="0 0 0"/>
-        <geometry>
-          <box size="${body_length} ${body_width} ${body_height}"/>
-        </geometry>
-      </collision>
-      <inertial>
-        <mass value="5.0"/>
-        <inertia
-           ixx="${1/12 * 5.0*(body_width*body_width+body_height*body_height)}"
-           ixy="0" ixz="0"
-           iyy="${1/12 * 5.0*(body_length*body_length+body_height*body_height)}"
-           iyz="0"
-           izz="${1/12 * 5.0*(body_length*body_length+body_width*body_width)}"/>
-      </inertial>
-    </link>
+  <!-- BASE LINK -->
+  <link name="base_link"/>
+  <!-- CHASSIS -->
+  <joint name="chassis_joint" type="fixed">
+    <parent link="base_link"/>
+    <child link="chassis"/>
+    <origin xyz="0 0 0.2"/>
+  </joint>
+  <link name="chassis">
+    <visual>
+      <origin xyz="0 0 0"/>
+      <geometry>
+        <box size="${body_length} ${body_width} ${body_height}"/>
+      </geometry>
+      <material name="grey"/>
+    </visual>
+    <collision>
+      <origin xyz="0 0 0"/>
+      <geometry>
+        <box size="${body_length} ${body_width} ${body_height}"/>
+      </geometry>
+    </collision>
+    <inertial>
+      <mass value="5.0"/>
+      <inertia
+         ixx="${1/12 * 5.0*(body_width*body_width+body_height*body_height)}"
+         ixy="0" ixz="0"
+         iyy="${1/12 * 5.0*(body_length*body_length+body_height*body_height)}"
+         iyz="0"
+         izz="${1/12 * 5.0*(body_length*body_length+body_width*body_width)}"/>
+    </inertial>
+  </link>
+  <!-- WHEEL MACRO -->
   <xacro:macro name="wheel" params="name x y">
     <joint name="base_${name}_joint" type="continuous">
@@ -73,10 +78,10 @@
       <inertial>
         <mass value="0.5"/>
-          <inertia
-             ixx="${(1/12) * 0.5 * (3*wheel_radius*wheel_radius+wheel_length*wheel_length)}"
-             ixy="0" ixz="0"
-             izz="${(1/2) * 0.5* (wheel_radius*wheel_radius)}"
-             iyz="0"
-             iyy="${(1/12) * 0.5 * (3*wheel_radius*wheel_radius+wheel_length*wheel_length)}"/>
+        <inertia
+           ixx="${(1/12) * 0.5 * (3*wheel_radius*wheel_radius+wheel_length*wheel_length)}"
+           ixy="0" ixz="0"
+           izz="${(1/2) * 0.5 * (wheel_radius*wheel_radius)}"
+           iyz="0"
+           iyy="${(1/12) * 0.5 * (3*wheel_radius*wheel_radius+wheel_length*wheel_length)}"/>
       </inertial>
     </link>
@@ -86,4 +91,29 @@
   <xacro:wheel name="right_front_wheel" x="${wheel_x}"  y="-${wheel_y}"/>
   <xacro:wheel name="right_back_wheel"  x="-${wheel_x}" y="-${wheel_y}"/>
+  <!-- LIDAR -->
+  <joint name="lidar_joint" type="fixed">
+    <parent link="chassis"/>
+    <child link="lidar_link"/>
+    <origin xyz="0 0 0.12"/>
+  </joint>
+  <link name="lidar_link">
+    <visual>
+      <geometry>
+        <cylinder radius="0.05" length="0.04"/>
+      </geometry>
+      <material name="black"/>
+    </visual>
+    <collision>
+      <geometry>
+        <cylinder radius="0.05" length="0.04"/>
+      </geometry>
+    </collision>
+    <inertial>
+      <mass value="0.1"/>
+      <inertia ixx="0.001" ixy="0" ixz="0"
+               iyy="0.001" iyz="0" izz="0.001"/>
+    </inertial>
+  </link>
+  <!-- DIFF DRIVE PLUGIN -->
   <gazebo>
     <plugin

Commit message: Nav2 params + map + EKF + IMU + fixed robot model. Foundation complete, ready for Nav2 bringup.

File: description/robot.urdf.xacro (robot description, xacro)
@@ -7,19 +7,10 @@
   <xacro:property name="wheel_radius" value="0.1"/>
   <xacro:property name="wheel_length" value="0.05"/>
-  <xacro:property name="wheel_x"      value="0.15"/>
-  <xacro:property name="wheel_y"      value="0.225"/>
+  <xacro:property name="wheel_x"      value="0.12"/>   <!-- short wheelbase: easier turning -->
+  <xacro:property name="wheel_y"      value="0.225"/>  <!-- half of separation 0.45 -->
   <!-- Materials -->
-  <material name="grey">
-    <color rgba="0.5 0.5 0.5 1"/>
-  </material>
-  <material name="blue">
-    <color rgba="0.1 0.1 0.8 1"/>
-  </material>
-  <material name="white">
-    <color rgba="1 1 1 1"/>
-  </material>
-  <material name="black">
-    <color rgba="0.1 0.1 0.1 1"/>
-  </material>
+  <material name="grey"><color rgba="0.5 0.5 0.5 1"/></material>
+  <material name="blue"><color rgba="0.1 0.1 0.8 1"/></material>
+  <material name="black"><color rgba="0.1 0.1 0.1 1"/></material>
   <!-- BASE LINK -->
   <link name="base_link"/>
@@ -33,14 +24,10 @@
     <visual>
       <origin xyz="0 0 0"/>
-      <geometry>
-        <box size="${body_length} ${body_width} ${body_height}"/>
-      </geometry>
+      <geometry><box size="${body_length} ${body_width} ${body_height}"/></geometry>
       <material name="grey"/>
     </visual>
     <collision>
       <origin xyz="0 0 0"/>
-      <geometry>
-        <box size="${body_length} ${body_width} ${body_height}"/>
-      </geometry>
+      <geometry><box size="${body_length} ${body_width} ${body_height}"/></geometry>
     </collision>
     <inertial>
@@ -54,7 +41,7 @@
     </inertial>
   </link>
-  <!-- WHEEL MACRO -->
+  <!-- WHEEL MACRO — skid-steer tuned (low lateral friction) -->
   <xacro:macro name="wheel" params="name x y">
-    <joint name="base_${name}_joint" type="continuous">
+    <joint name="${name}_joint" type="continuous">
       <parent link="chassis"/>
       <child link="${name}_link"/>
@@ -65,26 +52,31 @@
       <visual>
         <origin xyz="0 0 0" rpy="1.5708 0 0"/>
-        <geometry>
-          <cylinder radius="${wheel_radius}" length="${wheel_length}"/>
-        </geometry>
-        <material name="blue"/>
+        <geometry><cylinder radius="${wheel_radius}" length="${wheel_length}"/></geometry>
+        <material name="black"/>
       </visual>
       <collision>
         <origin xyz="0 0 0" rpy="1.5708 0 0"/>
-        <geometry>
-          <cylinder radius="${wheel_radius}" length="${wheel_length}"/>
-        </geometry>
+        <geometry><cylinder radius="${wheel_radius}" length="${wheel_length}"/></geometry>
       </collision>
       <inertial>
         <mass value="0.5"/>
         <inertia
-           ixx="${(1/12) * 0.5 * (3*wheel_radius*wheel_radius+wheel_length*wheel_length)}"
+           ixx="${(1/12)*0.5*(3*wheel_radius*wheel_radius+wheel_length*wheel_length)}"
            ixy="0" ixz="0"
-           izz="${(1/2) * 0.5 * (wheel_radius*wheel_radius)}"
+           iyy="${(1/12)*0.5*(3*wheel_radius*wheel_radius+wheel_length*wheel_length)}"
            iyz="0"
-           iyy="${(1/12) * 0.5 * (3*wheel_radius*wheel_radius+wheel_length*wheel_length)}"/>
+           izz="${(1/2)*0.5*(wheel_radius*wheel_radius)}"/>
       </inertial>
     </link>
+    <!-- KEY: mu1 high (drive grip), mu2 ZERO (free sideways slip for skid-steer) -->
+    <gazebo reference="${name}_link">
+      <mu1>1.0</mu1>
+      <mu2>0.0</mu2>
+      <kp>1000000.0</kp>
+      <kd>100.0</kd>
+      <fdir1>1 0 0</fdir1>
+    </gazebo>
   </xacro:macro>
+  <!-- Four driven wheels at the corners -->
   <xacro:wheel name="left_front_wheel"  x="${wheel_x}"  y="${wheel_y}"/>
   <xacro:wheel name="left_back_wheel"   x="-${wheel_x}" y="${wheel_y}"/>
@@ -99,21 +91,15 @@
   <link name="lidar_link">
     <visual>
-      <geometry>
-        <cylinder radius="0.05" length="0.04"/>
-      </geometry>
+      <geometry><cylinder radius="0.05" length="0.04"/></geometry>
       <material name="black"/>
     </visual>
     <collision>
-      <geometry>
-        <cylinder radius="0.05" length="0.04"/>
-      </geometry>
+      <geometry><cylinder radius="0.05" length="0.04"/></geometry>
     </collision>
     <inertial>
       <mass value="0.1"/>
-      <inertia ixx="0.001" ixy="0" ixz="0"
-               iyy="0.001" iyz="0" izz="0.001"/>
+      <inertia ixx="0.001" ixy="0" ixz="0" iyy="0.001" iyz="0" izz="0.001"/>
     </inertial>
   </link>
-  <!-- LIDAR SENSOR (Gazebo Fortress) -->
   <gazebo reference="lidar_link">
     <sensor name="lidar_sensor" type="gpu_lidar">
@@ -140,13 +126,27 @@
     </sensor>
   </gazebo>
-  <!-- DIFF DRIVE PLUGIN -->
+  <!-- IMU SENSOR -->
+  <gazebo reference="chassis">
+    <sensor name="imu_sensor" type="imu">
+      <topic>imu</topic>
+      <update_rate>50</update_rate>
+      <always_on>true</always_on>
+      <gz_frame_id>chassis</gz_frame_id>
+    </sensor>
+  </gazebo>
+  <!-- IMU SYSTEM PLUGIN — required for IMU to publish -->
   <gazebo>
-    <plugin
-       filename="ignition-gazebo-diff-drive-system"
-       name="ignition::gazebo::systems::DiffDrive">
-       <left_joint>base_left_front_wheel_joint</left_joint>
-       <left_joint>base_left_back_wheel_joint</left_joint>
-       <right_joint>base_right_front_wheel_joint</right_joint>
-       <right_joint>base_right_back_wheel_joint</right_joint>
+    <plugin filename="ignition-gazebo-imu-system"
+            name="ignition::gazebo::systems::Imu">
+    </plugin>
+  </gazebo>
+  <!-- DIFF DRIVE — all 4 wheels (2 left, 2 right) -->
+  <gazebo>
+    <plugin filename="ignition-gazebo-diff-drive-system"
+            name="ignition::gazebo::systems::DiffDrive">
+       <left_joint>left_front_wheel_joint</left_joint>
+       <left_joint>left_back_wheel_joint</left_joint>
+       <right_joint>right_front_wheel_joint</right_joint>
+       <right_joint>right_back_wheel_joint</right_joint>
        <wheel_separation>0.45</wheel_separation>
        <wheel_radius>${wheel_radius}</wheel_radius>
@@ -156,12 +156,17 @@
        <child_frame_id>base_link</child_frame_id>
        <publish_odom>true</publish_odom>
-       <publish_odom_tf>true</publish_odom_tf>
+       <publish_odom_tf>false</publish_odom_tf>
     </plugin>
   </gazebo>
-  <!-- SENSORS SYSTEM PLUGIN — required for lidar to publish data -->
+  <!-- JOINT STATE PUBLISHER — makes Gazebo publish wheel joint states -->
   <gazebo>
-    <plugin
-       filename="ignition-gazebo-sensors-system"
-       name="ignition::gazebo::systems::Sensors">
+    <plugin filename="ignition-gazebo-joint-state-publisher-system"
+            name="ignition::gazebo::systems::JointStatePublisher">
+    </plugin>
+  </gazebo>
+  <!-- SENSORS SYSTEM PLUGIN -->
+  <gazebo>
+    <plugin filename="ignition-gazebo-sensors-system"
+            name="ignition::gazebo::systems::Sensors">
        <render_engine>ogre2</render_engine>
     </plugin>
